File: emu6802.kicad5/emu6802/emu6802.sch (KiCad schematic (older format))
At the start: 20 parts, among them CON1 Conn_01x08, CON2 Conn_01x06, J3 Barrel_Jack_Switch, U1 PIC18F47Q84-DIP40, U2 MC6802

Commit message: update readme
Connections:
- net CLC2_G3POL: now also UX4.4 (R); no longer UX4.6 (S)
- net GND: now also UX4.6 (S); no longer UX4.4 (R)
Other:
- moved on the sheet: UX2A, UX4A
Changed lines of the file:
@@
 L 4xxx:4013 UX4
 U 1 1 62EFFDB6
-P 9700 4400
-F 0 "UX4" H 9850 4750 50  0000 C CNN
-F 1 "CLC2" H 9700 4400 50  0000 C CNN
-F 2 "" H 9700 4400 50  0001 C CNN
-F 3 "http://www.onsemi.com/pub/Collateral/MC14013B-D.PDF" H 9700 4400 50  0001 C CNN
-	1    9700 4400
+P 9700 3950
+F 0 "UX4" H 9850 4300 50  0000 C CNN
+F 1 "CLC2" H 9700 3950 50  0000 C CNN
+F 2 "" H 9700 3950 50  0001 C CNN
+F 3 "http://www.onsemi.com/pub/Collateral/MC14013B-D.PDF" H 9700 3950 50  0001 C CNN
+	1    9700 3950
 	1    0    0    -1
 $EndComp
@@
 	9250 2700 9150 2700
 Wire Wire Line
-	10000 4300 10150 4300
-Text GLabel 10150 4300 2    50   Input ~ 0
+	10000 3850 10150 3850
+Text GLabel 10150 3850 2    50   Input ~ 0
 RA2
 $Comp
 L 74xx:74LS04 UX2
 U 1 1 62F26A3E
-P 9000 4550
-F 0 "UX2" H 8950 4400 50  0000 C CNN
-F 1 "CLC1" H 8950 4550 50  0000 C CNN
-F 2 "" H 9000 4550 50  0001 C CNN
-F 3 "http://www.ti.com/lit/gpn/sn74LS04" H 9000 4550 50  0001 C CNN
-	1    9000 4550
+P 9000 4100
+F 0 "UX2" H 8950 3950 50  0000 C CNN
+F 1 "CLC1" H 8950 4100 50  0000 C CNN
+F 2 "" H 9000 4100 50  0001 C CNN
+F 3 "http://www.ti.com/lit/gpn/sn74LS04" H 9000 4100 50  0001 C CNN
+	1    9000 4100
 	1    0    0    -1
 $EndComp
 Wire Wire Line
-	9400 4400 9300 4400
+	9400 3950 9300 3950
 Wire Wire Line
-	9300 4400 9300 4550
-Text GLabel 8650 4550 0    50   Input ~ 0
+	9300 3950 9300 4100
+Text GLabel 8650 4100 0    50   Input ~ 0
 NCO1_OUT
 Text GLabel 8400 2700 0    50   Input ~ 0
@@
 Wire Wire Line
 	9850 2800 9950 2800
-Text GLabel 8750 4300 0    50   Input ~ 0
+Text GLabel 8750 3850 0    50   Input ~ 0
 CLC2_G2POL
 Wire Wire Line
-	8750 4300 9400 4300
-Text GLabel 8750 4000 0    50   Input ~ 0
+	8750 3850 9400 3850
+Text GLabel 8750 4400 0    50   Input ~ 0
 CLC2_G3POL
 Wire Wire Line
-	9700 4100 9700 4000
-Wire Wire Line
-	9700 4000 8750 4000
+	9700 4400 8750 4400
 $Comp
 L power:GND #PWR018
 U 1 1 62F727F3
-P 9700 4700
-F 0 "#PWR018" H 9700 4450 50  0001 C CNN
-F 1 "GND" H 9705 4527 50  0000 C CNN
-F 2 "" H 9700 4700 50  0001 C CNN
-F 3 "" H 9700 4700 50  0001 C CNN
-	1    9700 4700
+P 9500 3500
+F 0 "#PWR018" H 9500 3250 50  0001 C CNN
+F 1 "GND" H 9505 3327 50  0000 C CNN
+F 2 "" H 9500 3500 50  0001 C CNN
+F 3 "" H 9500 3500 50  0001 C CNN
+	1    9500 3500
 	1    0    0    -1
 $EndComp
-NoConn ~ 10000 4500
-Text Notes 7800 4350 0    50   ~ 0
+NoConn ~ 10000 4050
+Text Notes 7800 3900 0    50   ~ 0
 MPU_MRDY
-Text Notes 7750 4600 0    50   ~ 0
+Text Notes 7750 4150 0    50   ~ 0
 MPU_EXTAL
-Text Notes 7700 4050 0    50   ~ 0
+Text Notes 7700 4450 0    50   ~ 0
 MRDY_FF_RES
 Text Notes 7500 2200 0    94   ~ 0
 CLC1
-Text Notes 7500 3650 0    94   ~ 0
+Text Notes 7500 3500 0    94   ~ 0
 CLC2
 Text Notes 7500 5150 0    94   ~ 0
 NCO1
-Text Notes 10400 4350 0    50   ~ 0
+Text Notes 10400 3900 0    50   ~ 0
 MPU_MR
 Text Notes 7900 2750 0    50   ~ 0
@@
 	9000 5550 8850 5550
 Wire Wire Line
-	8700 4550 8650 4550
+	8700 4100 8650 4100
 Text Notes 9650 5550 0    50   ~ 0
 MPU_EXTAL
 Text Notes 7550 7500 0    50   ~ 0
 EMU6802, derived from EMUZ80
+Wire Wire Line
+	9700 4400 9700 4250
+Wire Wire Line
+	9700 3500 9500 3500
+Wire Wire Line
+	9700 3500 9700 3650
 $EndSCHEMATC

Commit message: update readmes
Connections:
- net +5V: now also U2.36 (RE)
- net GND: no longer U2.36 (RE)
Other:
- note added: "* ENABLE INT SRAM"
Changed lines of the file:
@@
 	4450 4350 4750 4350
 Connection ~ 4750 4350
-$Comp
-L power:GND #PWR014
-U 1 1 62D80B10
-P 4450 4450
-F 0 "#PWR014" H 4450 4200 50  0001 C CNN
-F 1 "GND" H 4455 4277 50  0000 C CNN
-F 2 "" H 4450 4450 50  0001 C CNN
-F 3 "" H 4450 4450 50  0001 C CNN
-	1    4450 4450
-	1    0    0    -1
-$EndComp
-Wire Wire Line
-	4600 4450 4450 4450
-Wire Wire Line
-	4600 4550 4750 4550
-Wire Wire Line
-	4600 4450 4600 4550
 NoConn ~ 5750 4650
 NoConn ~ 3650 4750
@@
 Wire Wire Line
 	9700 3500 9700 3650
+Wire Wire Line
+	4450 4550 4450 4350
+Wire Wire Line
+	4450 4550 4750 4550
+Connection ~ 4450 4350
+Text Notes 4000 4650 0    50   ~ 0
+* ENABLE INT SRAM
 $EndSCHEMATC
